File: design/blackpill_CNC_BoB.kicad_pcb (KiCad board)
At the start: 4 copper layers, 100 x 100 mm, 308 parts, among them J101 ALimIN, J102 ZLimIN, J103 YLimIN, J104 XLimIN, J105 CS_IN, J106 FH_IN, J107 DoorIN, J108 ResetIN, J109 ProbeIN, J110 12V Power in, J111 AuxEncIn, J112 5V Power out, J113 ADC_in_1, J114 ADC_in_2, J115 stepDriverLim, J116 Reset, J117 UART1, J118 I2C, J119 SpindleVFD, J120 Spindle/Coolant, J121 Spindle, J122 Coolant, J123 AuxOut, J124 XStepDrv, J125 YStepDrv, J126 ZStepDrv, J127 AStepDrv, J128 Driver Power in/out, J129 Relais Power in/out, J130 Conn_02x03_Odd_Even, J131 Conn_02x03_Odd_Even, U101 TLP290-4, U102 TLP290-4, U103 TLP290-4, U104 74LVC2G17, U105 LD1117S50TR_SOT223, U106 LM358, U107 TLV9001, U108 TLV9001, U109 YAAJ_WeAct_BlackPill_Part_Like, U110 TLV9001, U111 TLV9001, U112 74HCT541, U113 74HCT541, U114 74HCT541, U115 ULN2003A, U116 ULN2003A, U117 ULN2003A

Commit message: add 3.3 and 5V planes
Routing:
- added copper zone on In2.Cu, net (none)
- added copper zone on In2.Cu, net +3V3
- added copper zone on In2.Cu, net +5V
- added copper zone on In1.Cu, net GND
Changed lines of the file:
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@@
   (layers
     (0 F.Cu signal)
-    (1 In1.Cu signal)
+    (1 In1.Cu signal hide)
     (2 In2.Cu signal)
     (31 B.Cu signal)
@@
   (gr_line (start 100 0) (end 100 100) (layer Dwgs.User) (width 0.1))
   (gr_line (start 0 0) (end 100 0) (layer Dwgs.User) (width 0.1))
+  (zone (net 2) (net_name GND) (layer In1.Cu) (hatch edge 0.508)
+    (connect_pads (clearance 0.508))
+    (min_thickness 0.254)
+    (fill yes (arc_segments 32) (thermal_gap 0.508) (thermal_bridge_width 0.508))
+    (polygon
+      (pts
+        (xy 111.76 107.315) (xy -10.795 107.315) (xy -10.795 -6.985) (xy 111.76 -6.985)
+      )
+    )
+  )
+  (zone (net 1) (net_name +5V) (layer In2.Cu) (hatch edge 0.508)
+    (connect_pads (clearance 0.508))
+    (min_thickness 0.254)
+    (fill yes (arc_segments 32) (thermal_gap 0.508) (thermal_bridge_width 0.508))
+    (polygon
+      (pts
+        (xy 103.505 33.02) (xy -6.35 33.02) (xy -6.35 -1.905) (xy 103.505 -1.905)
+      )
+    )
+  )
+  (zone (net 4) (net_name +3V3) (layer In2.Cu) (hatch edge 0.508)
+    (connect_pads (clearance 0.508))
+    (min_thickness 0.254)
+    (fill yes (arc_segments 32) (thermal_gap 0.508) (thermal_bridge_width 0.508))
+    (polygon
+      (pts
+        (xy 62.23 106.045) (xy -7.62 106.68) (xy -5.715 74.93) (xy 60.96 74.93)
+      )
+    )
+  )
+  (zone (net 4) (net_name +3V3) (layer In2.Cu) (hatch edge 0.508)
+    (connect_pads (clearance 0.508))
+    (min_thickness 0.254)
+    (fill yes (arc_segments 32) (thermal_gap 0.508) (thermal_bridge_width 0.508))
+    (polygon
+      (pts
+        (xy -7.62 54.61) (xy 60.325 53.975) (xy 62.865 78.74) (xy -10.16 78.105) (xy -10.16 53.34)
+      )
+    )
+  )
+  (zone (net 0) (net_name "") (layer In2.Cu) (hatch edge 0.508)
+    (connect_pads (clearance 0.508))
+    (min_thickness 0.254)
+    (fill yes (arc_segments 32) (thermal_gap 0.508) (thermal_bridge_width 0.508))
+    (polygon
+      (pts
+        (xy 61.595 81.915) (xy -8.89 81.915) (xy -8.89 43.815) (xy 61.595 43.815)
+      )
+    )
+  )
+  (zone (net 0) (net_name "") (layer In2.Cu) (hatch edge 0.508)
+    (connect_pads (clearance 0.508))
+    (min_thickness 0.254)
+    (fill yes (arc_segments 32) (thermal_gap 0.508) (thermal_bridge_width 0.508))
+  )
+  (zone (net 4) (net_name +3V3) (layer In2.Cu) (hatch edge 0.508)
+    (connect_pads (clearance 0.508))
+    (min_thickness 0.254)
+    (fill yes (arc_segments 32) (thermal_gap 0.508) (thermal_bridge_width 0.508))
+    (polygon
+      (pts
+        (xy 62.865 47.625) (xy -12.065 47.625) (xy -12.065 41.91) (xy 62.865 41.91)
+      )
+    )
+  )
+  (zone (net 4) (net_name +3V3) (layer In2.Cu) (hatch edge 0.508)
+    (connect_pads (clearance 0.508))
+    (min_thickness 0.254)
+    (fill yes (arc_segments 32) (thermal_gap 0.508) (thermal_bridge_width 0.508))
+    (polygon
+      (pts
+        (xy 72.39 46.355) (xy 57.785 46.355) (xy 57.785 41.91) (xy 72.39 41.91)
+      )
+    )
+  )
+  (zone (net 4) (net_name +3V3) (layer In2.Cu) (hatch edge 0.508)
+    (connect_pads (clearance 0.508))
+    (min_thickness 0.254)
+    (fill yes (arc_segments 32) (thermal_gap 0.508) (thermal_bridge_width 0.508))
+  )
+  (zone (net 4) (net_name +3V3) (layer In2.Cu) (hatch edge 0.508)
+    (connect_pads (clearance 0.508))
+    (min_thickness 0.254)
+    (fill yes (arc_segments 32) (thermal_gap 0.508) (thermal_bridge_width 0.508))
+    (polygon
+      (pts
+        (xy 39.37 45.72) (xy -13.335 45.72) (xy -13.335 36.83) (xy 39.37 36.83)
+      )
+    )
+  )
+  (zone (net 4) (net_name +3V3) (layer In2.Cu) (hatch edge 0.508)
+    (connect_pads (clearance 0.508))
+    (min_thickness 0.254)
+    (fill yes (arc_segments 32) (thermal_gap 0.508) (thermal_bridge_width 0.508))
+    (polygon
+      (pts
+        (xy 12.065 39.37) (xy -2.54 39.37) (xy -2.54 36.195) (xy 12.065 36.195)
+      )
+    )
+  )
+  (zone (net 4) (net_name +3V3) (layer In2.Cu) (hatch edge 0.508)
+    (connect_pads (clearance 0.508))
+    (min_thickness 0.254)
+    (fill yes (arc_segments 32) (thermal_gap 0.508) (thermal_bridge_width 0.508))
+    (polygon
+      (pts
+        (xy 27.94 39.37) (xy 10.16 39.37) (xy 10.16 34.29) (xy 27.94 34.29)
+      )
+    )
+  )
 )

Commit message: routing...
Parts:
- moved D107 0.90 mm to (76.6, 80.4)
- moved D103 0.90 mm to (83.9, 80.4)
- moved D105 0.89 mm to (80.3, 80.4)
- moved C108 0.63 mm to (27.3, 33.7)
Routing:
- net GND: track 0.00 -> 283.3 mm, vias 0 -> 72
- net +5V: track 0.00 -> 78.5 mm, vias 0 -> 15
- net +3V3: track 0.00 -> 48.5 mm, vias 0 -> 7
- net /V_Drive: track 0.00 -> 46.6 mm
- net /V_relais: track 0.00 -> 46.6 mm
- net +12V: track 0.00 -> 46.0 mm
- net Net-(JP213-Pad2): track 0.00 -> 21.8 mm
- net Net-(JP219-Pad2): track 0.00 -> 21.0 mm
- net /AuxO1V: track 0.00 -> 20.7 mm
- net Net-(D106-Pad3): track 0.00 -> 19.7 mm
- net Net-(J104-Pad2): track 0.00 -> 18.9 mm
- net Net-(JP220-Pad1): track 0.00 -> 18.6 mm
- net Net-(JP104-Pad1): track 0.00 -> 18.4 mm
- net Net-(J103-Pad2): track 0.00 -> 18.1 mm
- net /FloodL: track 0.00 -> 17.9 mm
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
Commit message: routed front as possible...
Routing:
- net /SCL: track 0.00 -> 20.1 mm
- net /U5uC: track 0.00 -> 20.1 mm
- net Net-(JP153-Pad2): track 5.08 -> 22.2 mm
- net /YEnable: track 0.00 -> 16.5 mm
- net /XEnable: track 0.00 -> 15.4 mm
- net +3V3: track 48.5 -> 63.2 mm, vias 7 -> 6
- net /~Strobe: track 0.00 -> 14.5 mm
- net Net-(JP154-Pad2): track 2.54 -> 16.3 mm
- net Net-(JP158-Pad2): track 7.62 -> 19.8 mm
- net Net-(R101-Pad2): track 0.00 -> 10.6 mm
- net Net-(R102-Pad2): track 0.00 -> 9.89 mm
- net Net-(D120-Pad1): track 0.00 -> 9.35 mm
- net /SDA: track 0.00 -> 8.78 mm
- net GND: track 283.3 -> 288.7 mm
- net /Y_lim: track 0.00 -> 5.13 mm
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
Commit message: starte routing backside
Routing:
- net Net-(J109-Pad2): track 0.00 -> 38.0 mm, vias 0 -> 1
- net Net-(J108-Pad2): track 0.00 -> 35.3 mm, vias 0 -> 1
- net Net-(J107-Pad2): track 0.00 -> 32.6 mm, vias 0 -> 1
- net Net-(J106-Pad2): track 0.00 -> 29.1 mm, vias 0 -> 1
- net Net-(R109-Pad2): track 0.00 -> 27.6 mm, vias 0 -> 2
- net /XLim: track 7.85 -> 33.9 mm, vias 0 -> 1
- net Net-(J105-Pad2): track 0.00 -> 26.0 mm, vias 0 -> 1
- net /YLim: track 8.10 -> 29.7 mm, vias 0 -> 1
- net +5V: track 83.4 -> 102.8 mm, vias 15 -> 17
- net /ZLim: track 8.15 -> 24.5 mm, vias 0 -> 1
- net /ALim: track 8.11 -> 21.2 mm, vias 0 -> 1
- net Net-(JP142-Pad1): track 0.00 -> 6.72 mm
- net Net-(JP139-Pad2): track 0.00 -> 4.77 mm
- net Net-(JP138-Pad2): track 0.00 -> 3.50 mm
- net /AuxIn2: vias 0 -> 1
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
Commit message: simple stuff done
Routing:
- net +5V: track 102.8 -> 221.2 mm, vias 17 -> 25
- net +12V: track 46.0 -> 142.2 mm, vias 0 -> 1
- net /V_Drive: track 46.6 -> 116.7 mm, vias 0 -> 1
- net /SDA: track 8.78 -> 71.4 mm, vias 0 -> 1
- net /SCL: track 20.1 -> 73.3 mm, vias 0 -> 1
- net /AuxIn1: track 0.00 -> 50.3 mm, vias 0 -> 1
- net /AuxIn0: track 0.00 -> 46.9 mm, vias 0 -> 1
- net Net-(JP99-Pad1): track 0.00 -> 40.0 mm, vias 0 -> 3
- net /V_relais: track 46.6 -> 86.2 mm
- net /AuxO0V: track 0.00 -> 38.0 mm, vias 0 -> 1
- net /ZEnable: track 0.00 -> 36.2 mm, vias 0 -> 1
- net /AEnable: track 0.00 -> 34.8 mm, vias 0 -> 1
- net /AuxIn2: track 2.91 -> 32.2 mm
- net /YDir: track 0.00 -> 28.2 mm, vias 0 -> 1
- net /YStep: track 0.00 -> 24.9 mm, vias 0 -> 1
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
Commit message: routing diff power
Routing:
- net +3V3: track 83.6 -> 126.8 mm, vias 7 -> 8
- net /UADCdriver: track 14.2 -> 45.9 mm, vias 0 -> 2
- net +5V: track 221.2 -> 248.4 mm
- net /SPenO: track 12.4 -> 31.8 mm
- net Net-(J114-Pad2): track 0.00 -> 17.7 mm
- net /SPdirO: track 11.5 -> 28.0 mm
- net /MistL: track 11.9 -> 25.4 mm
- net +12V: track 142.2 -> 141.3 mm, vias 1 -> 8

Commit message: routing bot right
Routing:
- added copper zone on In2.Cu, net +12V
Changed lines of the file:
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@@
+    )
+  )
+  (zone (net 3) (net_name +12V) (layer In2.Cu) (hatch edge 0.508)
+    (connect_pads (clearance 0.508))
+    (min_thickness 0.254)
+    (fill yes (arc_segments 32) (thermal_gap 0.508) (thermal_bridge_width 0.508))
+    (polygon
+      (pts
+        (xy 100.965 35.687) (xy 100.965 102.87) (xy 89.535 102.87) (xy 89.535 35.433) (xy 101.219 35.433)
+      )
+    )
+  )
+  (zone (net 3) (net_name +12V) (layer In2.Cu) (hatch edge 0.508)
+    (connect_pads (clearance 0.508))
+    (min_thickness 0.254)
+    (fill yes (arc_segments 32) (thermal_gap 0.508) (thermal_bridge_width 0.508))
+    (polygon
+      (pts
+        (xy 90.17 102.997) (xy 78.74 102.997) (xy 78.74 85.852) (xy 85.217 85.852) (xy 90.17 80.899)
+      )
+    )
+  )
+  (zone (net 1) (net_name +5V) (layer In2.Cu) (hatch edge 0.508)
+    (connect_pads (clearance 0.508))
+    (min_thickness 0.254)
+    (fill yes (arc_segments 32) (thermal_gap 0.508) (thermal_bridge_width 0.508))
+    (polygon
+      (pts
+        (xy 87.884 40.894) (xy 40.259 40.894) (xy 40.259 32.385) (xy 87.884 32.385)
+      )
+    )
+  )
+  (zone (net 4) (net_name +3V3) (layer In2.Cu) (hatch edge 0.508)
+    (connect_pads (clearance 0.508))
+    (min_thickness 0.254)
+    (fill yes (arc_segments 32) (thermal_gap 0.508) (thermal_bridge_width 0.508))
+    (polygon
+      (pts
+        (xy 72.517 97.155) (xy 55.499 97.155) (xy 55.499 45.847) (xy 72.517 45.847)
+      )
+    )
+  )
+  (zone (net 1) (net_name +5V) (layer In2.Cu) (hatch edge 0.508)
+    (connect_pads (clearance 0.508))
+    (min_thickness 0.254)
+    (fill yes (arc_segments 32) (thermal_gap 0.508) (thermal_bridge_width 0.508))
+    (polygon
+      (pts
+        (xy 87.884 81.407) (xy 84.836 84.455) (xy 75.438 84.455) (xy 75.438 37.592) (xy 87.884 37.592)
+      )
+    )
+  )
+  (zone (net 1) (net_name +5V) (layer In2.Cu) (hatch edge 0.508)
+    (connect_pads (clearance 0.508))
+    (min_thickness 0.254)
+    (fill yes (arc_segments 32) (thermal_gap 0.508) (thermal_bridge_width 0.508))
+    (polygon
+      (pts
+        (xy 78.232 59.309) (xy 76.073 59.309) (xy 73.279 56.515) (xy 73.279 36.703) (xy 78.232 36.703)
+      )
+    )
+  )
+  (zone (net 4) (net_name +3V3) (layer In2.Cu) (hatch edge 0.508)
+    (connect_pads (clearance 0.508))
+    (min_thickness 0.254)
+    (fill yes (arc_segments 32) (thermal_gap 0.508) (thermal_bridge_width 0.508))
+    (polygon
+      (pts
+        (xy 76.327 97.028) (xy 71.247 97.028) (xy 71.247 86.487) (xy 76.327 86.487)
+      )
+    )
+  )
+  (zone (net 3) (net_name +12V) (layer In2.Cu) (hatch edge 0.508)
+    (connect_pads (clearance 0.508))
+    (min_thickness 0.254)
+    (fill yes (arc_segments 32) (thermal_gap 0.508) (thermal_bridge_width 0.508))
+    (polygon
+      (pts
+        (xy 81.026 99.441) (xy 77.343 99.441) (xy 77.343 85.725) (xy 81.026 85.725)
+      )
+    )
+  )
+  (zone (net 4) (net_name +3V3) (layer In2.Cu) (hatch edge 0.508)
+    (connect_pads (clearance 0.508))
+    (min_thickness 0.254)
+    (fill yes (arc_segments 32) (thermal_gap 0.508) (thermal_bridge_width 0.508))
+    (polygon
+      (pts
+        (xy 78.359 63.754) (xy 78.359 73.279) (xy 76.327 75.311) (xy 76.327 81.026) (xy 73.279 81.026)
+        (xy 71.755 82.55) (xy 71.755 58.928) (xy 71.374 58.928) (xy 71.12 58.674) (xy 73.279 58.674)
+      )
     )
   )

Commit message: tuning power plates
Routing:
- net +12V: track 141.3 -> 199.6 mm
- net /U5uC: track 20.1 -> 67.7 mm
- net +3V3: track 126.8 -> 146.5 mm, vias 8 -> 14
- net +5V: track 248.4 -> 267.4 mm
- net /V_relais: track 86.2 -> 97.6 mm
- net /V_Drive: track 116.7 -> 112.8 mm, vias 1 -> 0
- removed copper zone on In2.Cu, net (none)
