File: design/blackpill_CNC_BoB.sch (KiCad schematic (older format))
At the start: 308 parts, among them J101 ALimIN, J102 ZLimIN, J103 YLimIN, J104 XLimIN, J105 CS_IN, J106 FH_IN, J107 DoorIN, J108 ResetIN, J109 ProbeIN, J110 12V Power in, J111 AuxEncIn, J112 5V Power out, J113 ADC_in_1, J114 ADC_in_2, J115 stepDriverLim, J116 Reset, J117 UART1, J118 I2C, J119 SpindleVFD, J120 Spindle/Coolant, J121 Spindle, J122 Coolant, J123 AuxOut, J124 XStepDrv, J125 YStepDrv, J126 ZStepDrv, J127 AStepDrv, J128 Driver Power in/out, J129 Relais Power in/out, J130 Conn_02x03_Odd_Even, J131 Conn_02x03_Odd_Even, U101 TLP290-4, U102 TLP290-4, U103 TLP290-4, U104 74LVC2G17, U105 LD1117S50TR_SOT223, U106 LM358, U107 TLV9001, U108 TLV9001, U109 YAAJ_WeAct_BlackPill_Part_Like, U110 TLV9001, U111 TLV9001, U112 74HCT541, U113 74HCT541, U114 74HCT541, U115 ULN2003A, U116 ULN2003A, U117 ULN2003A

Commit message: DRC check after changes OK
Parts:
- C104: value 470µF -> 470uF
- C119: value 1µF -> 1uF
- C98: value 47µF -> 47uF
- C99: value 22µF -> 22uF
Changed lines of the file:
@@
 P 9000 10500
 F 0 "C119" H 9050 10400 50  0000 L CNN
-F 1 "1µF" H 8900 10600 50  0000 L CNN
+F 1 "1uF" H 8900 10600 50  0000 L CNN
 F 2 "Capacitor_SMD:C_0603_1608Metric" H 9038 10350 50  0001 C CNN
 F 3 "~" H 9000 10500 50  0001 C CNN
@@
 P 2950 10100
 F 0 "C104" H 2900 10000 50  0000 L CNN
-F 1 "470µF" H 2850 10250 50  0000 L CNN
+F 1 "470uF" H 2850 10250 50  0000 L CNN
 F 2 "Capacitor_SMD:CP_Elec_10x10" H 2988 9950 50  0001 C CNN
 F 3 "~" H 2950 10100 50  0001 C CNN
@@
 P 1950 10100
 F 0 "C99" H 1900 10000 50  0000 L CNN
-F 1 "22µF" H 1850 10250 50  0000 L CNN
+F 1 "22uF" H 1850 10250 50  0000 L CNN
 F 2 "Capacitor_SMD:C_1206_3216Metric" H 1988 9950 50  0001 C CNN
 F 3 "~" H 1950 10100 50  0001 C CNN
@@
 P 3200 10100
 F 0 "C98" H 3150 10000 50  0000 L CNN
-F 1 "47µF" H 3100 10200 50  0000 L CNN
+F 1 "47uF" H 3100 10200 50  0000 L CNN
 F 2 "Capacitor_SMD:C_1206_3216Metric" H 3238 9950 50  0001 C CNN
 F 3 "~" H 3200 10100 50  0001 C CNN
